Commit message: TEST COMPLETE

File: install/kuka_description/share/kuka_description/urdf/arduinobot.urdf.xacro (robot description, xacro)
@@ -1,176 +1 @@
-<?xml version="1.0"?>
-<robot xmlns:xacro="http://www.ros.org/wiki/xacro" name="arduinobot">
-    <!-- Useful XACRO Variables (Properties) -->
-    <xacro:property name="PI" value="3.14159265359" />
-    <xacro:property name="effort" value="30.0" />
-    <xacro:property name="velocity" value="10.0" />
-    <!-- Useful Macros -->
-    <xacro:macro name="default_inertial" params="mass">
-        <inertial>
-            <origin xyz="0 0 0" rpy="0 0 0"/>
-            <mass value="${mass}" />
-            <inertia ixx="1.0" ixy="0.0" ixz="0.0"
-                     iyy="1.0" iyz="0.0"
-                     izz="1.0" />
-        </inertial>
-    </xacro:macro>
-    <!-- Links -->
-    <link name="world"/>
-    <link name="base_link">
-        <xacro:default_inertial mass="1.0"/>
-        <visual>
-            <origin rpy="0 0 0" xyz="-0.5 -0.5 0"/>
-            <geometry>
-                <mesh filename="package://arduinobot_description/meshes/basement.STL" scale="0.01 0.01 0.01"/>
-            </geometry>
-        </visual>
-        <collision>
-            <origin rpy="0 0 0" xyz="-0.5 -0.5 0"/>
-            <geometry>
-                <mesh filename="package://arduinobot_description/meshes/basement.STL" scale="0.01 0.01 0.01"/>
-            </geometry>
-        </collision>
-    </link>
-    <link name="base_plate">
-        <xacro:default_inertial mass="0.1"/>
-        <visual>
-            <origin rpy="0 0 0" xyz="-0.39 -0.39 -0.56"/>
-            <geometry>
-                <mesh filename="package://arduinobot_description/meshes/base_plate.STL" scale="0.01 0.01 0.01"/>
-            </geometry>
-        </visual>
-        <collision>
-            <origin rpy="0 0 0" xyz="-0.39 -0.39 -0.56"/>
-            <geometry>
-                <mesh filename="package://arduinobot_description/meshes/base_plate.STL" scale="0.01 0.01 0.01"/>
-            </geometry>
-        </collision>
-    </link>
-    <link name="forward_drive_arm">
-        <xacro:default_inertial mass="0.1"/>
-        <visual>
-            <origin rpy=" 0 -${PI / 2} ${PI / 2}" xyz="0.19 0.06 -0.08"/>
-            <geometry>
-                <mesh filename="package://arduinobot_description/meshes/forward_drive_arm.STL" scale="0.01 0.01 0.01"/>
-            </geometry>
-        </visual>
-        <collision>
-            <origin rpy=" 0 -${PI / 2} ${PI / 2}" xyz="0.19 0.06 -0.08"/>
-            <geometry>
-                <mesh filename="package://arduinobot_description/meshes/forward_drive_arm.STL" scale="0.01 0.01 0.01"/>
-            </geometry>
-        </collision>
-    </link>
-    <link name="horizontal_arm">
-        <xacro:default_inertial mass="0.1"/>
-        <visual>
-            <origin rpy="${PI / 2} 0 ${PI / 2}" xyz="-0.03 -0.4 -0.06"/>
-            <geometry>
-                <mesh filename="package://arduinobot_description/meshes/horizontal_arm.STL" scale="0.01 0.01 0.01"/>
-            </geometry>
-        </visual>
-        <collision>
-            <origin rpy="${PI / 2} 0 ${PI / 2}" xyz="-0.03 -0.4 -0.06"/>
-            <geometry>
-                <mesh filename="package://arduinobot_description/meshes/horizontal_arm.STL" scale="0.01 0.01 0.01"/>
-            </geometry>
-        </collision>
-    </link>
-    <link name="claw_support">
-        <xacro:default_inertial mass="0.05"/>
-        <visual>
-            <origin rpy="0 0 ${PI / 2}" xyz="0 -0.05 -0.15"/>
-            <geometry>
-                <mesh filename="package://arduinobot_description/meshes/claw_support.STL" scale="0.01 0.01 0.01"/>
-            </geometry>
-        </visual>
-        <collision>
-            <origin rpy="0 0 ${PI / 2}" xyz="0 -0.05 -0.15"/>
-            <geometry>
-                <mesh filename="package://arduinobot_description/meshes/claw_support.STL" scale="0.01 0.01 0.01"/>
-            </geometry>
-        </collision>
-    </link>
-    <link name="gripper_right">
-        <xacro:default_inertial mass="0.01"/>
-        <visual>
-            <origin rpy="0 0 -${PI / 2}" xyz="-0.1 0.50 -0.1"/>
-            <geometry>
-                <mesh filename="package://arduinobot_description/meshes/right_finger.STL" scale="0.01 0.01 0.01"/>
-            </geometry>
-        </visual>
-        <collision>
-            <origin rpy="0 0 -${PI / 2}" xyz="-0.1 0.50 -0.1"/>
-            <geometry>
-                <mesh filename="package://arduinobot_description/meshes/right_finger.STL" scale="0.01 0.01 0.01"/>
-            </geometry>
-        </collision>
-    </link>
-    <link name="gripper_left">
-        <xacro:default_inertial mass="0.01"/>
-        <visual>
-            <origin rpy="0 0 -${PI / 2}" xyz="-0.04 0.50 -0.1"/>
-            <geometry>
-                <mesh filename="package://arduinobot_description/meshes/left_finger.STL" scale="0.01 0.01 0.01"/>
-            </geometry>
-        </visual>
-        <collision>
-            <origin rpy="0 0 -${PI / 2}" xyz="-0.04 0.50 -0.1"/>
-            <geometry>
-                <mesh filename="package://arduinobot_description/meshes/left_finger.STL" scale="0.01 0.01 0.01"/>
-            </geometry>
-        </collision>
-    </link>
-    <!-- Joints -->
-    <joint name="virtual_joint" type="fixed">
-        <parent link="world"/>
-        <child link="base_link"/>
-        <origin xyz="0 0 0" rpy="0 0 0"/>
-    </joint>
-    <joint name ="joint_1" type="revolute">
-        <parent link="base_link"/>
-        <child link = "base_plate"/>
-        <origin xyz="0 0 0.307"/>
-        <axis xyz="0 0 1"/>
-        <limit lower="-${PI / 2}" upper="${PI / 2}"
-               effort="${effort}" velocity="${velocity}"/>
-    </joint>
-    <joint name ="joint_2" type="revolute">
-        <parent link="base_plate"/>
-        <child link = "forward_drive_arm"/>
-        <origin xyz="-0.02 0 0.35"/>
-        <axis xyz="1 0 0"/>
-        <limit lower="-${PI / 2}" upper="${PI / 2}"
-                effort="${effort}" velocity="${velocity}"/>
-    </joint>
-    <joint name ="joint_3" type="revolute">
-        <parent link="forward_drive_arm"/>
-        <child link = "horizontal_arm"/>
-        <origin xyz="0 0 0.8"/>
-        <axis xyz="1 0 0"/>
-        <limit lower="-${PI / 2}" upper="${PI / 2}"
-               effort="${effort}" velocity="${velocity}"/>
-    </joint>
-    <joint name ="horizontal_arm_to_claw_support" type="fixed">
-        <parent link="horizontal_arm"/>
-        <child link = "claw_support"/>
-        <origin xyz="0 0.82 0"/>
-    </joint>
-    <joint name ="joint_4" type="revolute">
-        <parent link="claw_support"/>
-        <child link = "gripper_right"/>
-        <origin xyz="-0.04 0.13 -0.1"/>
-        <axis xyz="0 0 1"/>
-        <limit lower="-${PI / 2}" upper="0.0"
-               effort="${effort}" velocity="${velocity}"/>
-    </joint>
-    <joint name ="joint_5" type="revolute">
-        <parent link="claw_support"/>
-        <child link = "gripper_left"/>
-        <origin xyz="-0.22 0.13 -0.1"/>
-        <axis xyz="0 0 1"/>
-        <limit lower="0.0" upper="${PI / 2}"
-               effort="${effort}" velocity="${velocity}"/>
-        <mimic joint="joint_4" multiplier="-1"/>
-    </joint>
-</robot>
+/home/kuka/kuka_ws/src/kuka_description/urdf/arduinobot.urdf.xacro

File: install/kuka_description/share/kuka_description/urdf/kuka.urdf.xacro (robot description, xacro)
@@ -1,162 +1 @@
-<?xml version="1.0"?>
-<robot xmlns:xacro="http://www.ros.org/wiki/xacro" name="kuka">
-    <xacro:property name="PI" value="3.14159265359" />
-    <xacro:property name="DEG2RAD" value="0.01745329251" />
-    <xacro:property name="effort" value="30.0" />
-    <xacro:property name="velocity" value="10.0" />
-    <!-- Links -->
-    <link name="world"/>
-    <link name="base_link">
-        <visual>
-            <origin rpy="0 0 0" xyz="0 0 0"/>
-            <geometry>
-                <mesh filename="package://kuka_description/meshes/link0_exp.stl" scale="1 1 1"/>
-            </geometry>
-        </visual>
-        <collision>
-            <origin rpy="0 0 0" xyz="0 0 0"/>
-            <geometry>
-                <mesh filename="package://kuka_description/meshes/link0_exp.stl" scale="1 1 1"/>
-            </geometry>
-        </collision>
-    </link>
-    <link name="link_1">
-        <visual>
-            <origin rpy="${PI / 2} 0 ${PI}" xyz="0.33 0 0.67"/>
-            <geometry>
-                <mesh filename="package://kuka_description/meshes/link1_exp.stl" scale="1 1 1"/>
-            </geometry>
-        </visual>
-        <collision>
-            <origin rpy="${PI / 2} 0 ${PI}" xyz="0.33 0 0.67"/>
-            <geometry>
-                <mesh filename="package://kuka_description/meshes/link1_exp.stl" scale="1 1 1"/>
-            </geometry>
-        </collision>
-    </link>
-    <link name="link_2">
-        <visual>
-            <origin rpy="0 0 ${PI-2*DEG2RAD}" xyz="-1.176 -0.015 0.1"/>
-            <geometry>
-                <mesh filename="package://kuka_description/meshes/link2_exp.stl" scale="1 1 1"/>
-            </geometry>
-        </visual>
-        <collision>
-            <origin rpy="0 0 ${PI}" xyz="-1.176 -0.015 0.1"/>
-            <geometry>
-                <mesh filename="package://kuka_description/meshes/link2_exp.stl" scale="1 1 1"/>
-            </geometry>
-        </collision>
-    </link>
-    <link name="link_3">
-        <visual>
-            <origin rpy="${PI/2} 0 ${PI/2}" xyz="-0.03 -0.15 0.01"/>
-            <geometry>
-                <mesh filename="package://kuka_description/meshes/link3_exp.stl" scale="1 1 1"/>
-            </geometry>
-        </visual>
-        <collision>
-            <origin rpy="0 0 ${PI/2}" xyz="-0.03 -0.15 0.01"/>
-            <geometry>
-                <mesh filename="package://kuka_description/meshes/link3_exp.stl" scale="1 1 1"/>
-            </geometry>
-        </collision>
-    </link>
-    <link name="link_4">
-        <visual>
-            <origin rpy="${PI/2} 0 ${PI}" xyz="0 0 1.2"/>
-            <geometry>
-                <mesh filename="package://kuka_description/meshes/link4_exp.stl" scale="1 1 1"/>
-            </geometry>
-        </visual>
-        <collision>
-            <origin rpy="${PI/2} 0 ${PI}" xyz="0 0 1.2"/>
-            <geometry>
-                <mesh filename="package://kuka_description/meshes/link4_exp.stl" scale="1 1 1"/>
-            </geometry>
-        </collision>
-    </link>
-    <link name="link_5">
-        <visual>
-            <origin rpy="${PI/2} 0 ${PI}" xyz="0 -0.03 -0.01"/>
-            <geometry>
-                <mesh filename="package://kuka_description/meshes/link5_exp.stl" scale="1 1 1"/>
-            </geometry>
-        </visual>
-        <collision>
-            <origin rpy="${PI/2} 0 ${PI}" xyz="0 -0.03 -0.01"/>
-            <geometry>
-                <mesh filename="package://kuka_description/meshes/link5_exp.stl" scale="1 1 1"/>
-            </geometry>
-        </collision>
-    </link>
-    <link name="link_6">
-        <visual>
-            <origin rpy="${PI} 0 ${PI}" xyz="0 0 -0.02"/>
-            <geometry>
-                <mesh filename="package://kuka_description/meshes/link6_exp.stl" scale="1 1 1"/>
-            </geometry>
-        </visual>
-        <collision>
-            <origin rpy="${PI} 0 ${PI}" xyz="0 0 -0.02"/>
-            <geometry>
-                <mesh filename="package://kuka_description/meshes/link6_exp.stl" scale="1 1 1"/>
-            </geometry>
-        </collision>
-    </link>
-    <!-- Joints -->
-    <!-- Joint Limit Should be justified -->
-    <joint name="virtual_joint" type="fixed">
-        <parent link="world"/>
-        <child link="base_link"/>
-        <origin xyz="0 0 0" rpy="0 0 0"/>
-    </joint>
-    <joint name ="joint_1" type="revolute">
-        <parent link="base_link"/>
-        <child link = "link_1"/>
-        <origin xyz="0 0 0"/>
-        <axis xyz="0 0 1"/>
-        <limit lower="-${185*DEG2RAD}" upper="${185*DEG2RAD}"
-               effort="${effort}" velocity="${velocity}"/>
-    </joint>
-    <joint name ="joint_2" type="revolute">
-        <parent link="link_1"/>
-        <child link = "link_2"/>
-        <origin rpy="-${PI / 2} ${PI} 0" xyz="0.33 0 0.645"/>
-        <axis xyz="0 0 1"/>
-        <limit lower="-${140*DEG2RAD}" upper="-${5*DEG2RAD}"
-               effort="${effort}" velocity="${velocity}"/>
-    </joint>
-    <joint name ="joint_3" type="revolute">
-        <parent link="link_2"/>
-        <child link = "link_3"/>
-        <origin rpy="0 0 ${PI}" xyz="-1.150 0 0"/>
-        <axis xyz="0 0 1"/>
-        <limit lower="-${120*DEG2RAD}" upper="${168*DEG2RAD}"
-               effort="${effort}" velocity="${velocity}"/>
-    </joint>
-    <joint name ="joint_4" type="revolute">
-        <parent link="link_3"/>
-        <child link = "link_4"/>
-        <origin rpy="${PI/2} 0 ${PI/2}" xyz="0 -0.115 0"/>
-        <axis xyz="0 0 1"/>
-        <limit lower="-${350*DEG2RAD}" upper="${350*DEG2RAD}"
-               effort="${effort}" velocity="${velocity}"/>
-    </joint>
-    <joint name ="joint_5" type="revolute">
-        <parent link="link_4"/>
-        <child link = "link_5"/>
-        <origin rpy="${PI/2} 0 ${PI}" xyz="0 0 1.220"/>
-        <axis xyz="0 0 1"/>
-        <limit lower="-${122.5*DEG2RAD}" upper="${122.5*DEG2RAD}"
-               effort="${effort}" velocity="${velocity}"/>
-    </joint>
-    <joint name ="joint_6" type="revolute">
-        <parent link="link_5"/>
-        <child link = "link_6"/>
-        <origin rpy="${PI/2} 0 ${PI}" xyz="0 0.24 0"/>
-        <axis xyz="0 0 1"/>
-        <limit lower="-${350*DEG2RAD}" upper="${350*DEG2RAD}"
-               effort="${effort}" velocity="${velocity}"/>
-    </joint>
-</robot>
+/home/kuka/kuka_ws/src/kuka_description/urdf/kuka.urdf.xacro

File: src/kuka_description/urdf/kuka.urdf.xacro (robot description, xacro)
@@ -1,11 +1,34 @@
 <?xml version="1.0"?>
 <robot xmlns:xacro="http://www.ros.org/wiki/xacro" name="kuka">
+    <!-- Include Gazebo Parameters -->
+    <xacro:include filename="$(find kuka_description)/urdf/kuka_gazebo.xacro" />
+    <!-- Include ros2_control Plugins -->
+    <xacro:include filename="$(find kuka_description)/urdf/kuka_ros2_control.xacro" />
     <xacro:property name="PI" value="3.14159265359" />
     <xacro:property name="DEG2RAD" value="0.01745329251" />
     <xacro:property name="effort" value="30.0" />
     <xacro:property name="velocity" value="10.0" />
+    <xacro:macro name="default_inertial" params="mass">
+        <inertial>
+            <origin xyz="0 0 0" rpy="0 0 0"/>
+            <mass value="${mass}" />
+            <inertia ixx="1.0" ixy="0.0" ixz="0.0"
+                     iyy="1.0" iyz="0.0"
+                     izz="1.0" />
+        </inertial>
+    </xacro:macro>
+    <xacro:macro name="default_transmission" params="number">
+        <transmission name="transmission_${number}">
+            <plugin>transmission_interface/SimpleTransmission</plugin>
+            <actuator name="motor_${number}" role="actuator1"/>
+            <joint name="joint_${number}"    role="joint1">
+                <mechanical_reduction>1.0</mechanical_reduction>
+            </joint>
+        </transmission>
+    </xacro:macro>
     <!-- Links -->
     <link name="world"/>
     <link name="base_link">
+        <xacro:default_inertial mass="0.1"/>
         <visual>
             <origin rpy="0 0 0" xyz="0 0 0"/>
@@ -13,4 +36,7 @@
                 <mesh filename="package://kuka_description/meshes/link0_exp.stl" scale="1 1 1"/>
             </geometry>
+            <material name="">
+                <color rgba="0 0 0 1"/>
+            </material>
         </visual>
         <collision>
@@ -22,4 +48,5 @@
     </link>
     <link name="link_1">
+        <xacro:default_inertial mass="0.1"/>
         <visual>
             <origin rpy="${PI / 2} 0 ${PI}" xyz="0.33 0 0.67"/>
@@ -27,4 +54,7 @@
                 <mesh filename="package://kuka_description/meshes/link1_exp.stl" scale="1 1 1"/>
             </geometry>
+            <material name="">
+                <color rgba="0.9607 0.4117 0.0549 1"/>
+            </material>
         </visual>
         <collision>
@@ -36,4 +66,5 @@
     </link>
     <link name="link_2">
+        <xacro:default_inertial mass="0.1"/>
         <visual>
             <origin rpy="0 0 ${PI-2*DEG2RAD}" xyz="-1.176 -0.015 0.1"/>
@@ -41,4 +72,7 @@
                 <mesh filename="package://kuka_description/meshes/link2_exp.stl" scale="1 1 1"/>
             </geometry>
+            <material name="">
+                <color rgba="0.9607 0.4117 0.0549 1"/>
+            </material>
         </visual>
         <collision>
@@ -50,4 +84,5 @@
     </link>
     <link name="link_3">
+        <xacro:default_inertial mass="0.1"/>
         <visual>
             <origin rpy="${PI/2} 0 ${PI/2}" xyz="-0.03 -0.15 0.01"/>
@@ -55,4 +90,7 @@
                 <mesh filename="package://kuka_description/meshes/link3_exp.stl" scale="1 1 1"/>
             </geometry>
+            <material name="">
+                <color rgba="0.9607 0.4117 0.0549 1"/>
+            </material>
         </visual>
         <collision>
@@ -64,4 +102,5 @@
     </link>
     <link name="link_4">
+        <xacro:default_inertial mass="0.1"/>
         <visual>
             <origin rpy="${PI/2} 0 ${PI}" xyz="0 0 1.2"/>
@@ -69,4 +108,7 @@
                 <mesh filename="package://kuka_description/meshes/link4_exp.stl" scale="1 1 1"/>
             </geometry>
+            <material name="">
+                <color rgba="0.9607 0.4117 0.0549 1"/>
+            </material>
         </visual>
         <collision>
@@ -78,4 +120,5 @@
     </link>
     <link name="link_5">
+        <xacro:default_inertial mass="0.1"/>
         <visual>
             <origin rpy="${PI/2} 0 ${PI}" xyz="0 -0.03 -0.01"/>
@@ -83,4 +126,7 @@
                 <mesh filename="package://kuka_description/meshes/link5_exp.stl" scale="1 1 1"/>
             </geometry>
+            <material name="">
+                <color rgba="0.9607 0.4117 0.0549 1"/>
+            </material>
         </visual>
         <collision>
@@ -92,4 +138,5 @@
     </link>
     <link name="link_6">
+        <xacro:default_inertial mass="0.1"/>
         <visual>
             <origin rpy="${PI} 0 ${PI}" xyz="0 0 -0.02"/>
@@ -97,4 +144,7 @@
                 <mesh filename="package://kuka_description/meshes/link6_exp.stl" scale="1 1 1"/>
             </geometry>
+            <material name="">
+                <color rgba="0 0 0 1"/>
+            </material>
         </visual>
         <collision>
@@ -160,3 +210,10 @@
                effort="${effort}" velocity="${velocity}"/>
     </joint>
+    <!-- Transmissions-->
+    <xacro:default_transmission number="1"/>
+    <xacro:default_transmission number="2"/>
+    <xacro:default_transmission number="3"/>
+    <xacro:default_transmission number="4"/>
+    <xacro:default_transmission number="5"/>
+    <xacro:default_transmission number="6"/>
 </robot>
