Commit message: Add realsense-ros and apriltag_ros as submodules

File: src/kuka_description/urdf/kuka.urdf.xacro (robot description, xacro)
@@ -5,4 +5,5 @@
     <!-- Include ros2_control Plugins -->
     <xacro:include filename="$(find kuka_description)/urdf/kuka_ros2_control.xacro" />
+    <xacro:include filename="$(find kuka_description)/urdf/realsense_camera.xacro" />
     <xacro:property name="PI" value="3.14159265359" />
     <xacro:property name="DEG2RAD" value="0.01745329251" />
@@ -50,5 +51,5 @@
         <xacro:default_inertial mass="0.1"/>
         <visual>
-            <origin rpy="${PI / 2} 0 ${PI}" xyz="0.33 0 0.67"/>
+            <origin rpy="-${PI/2} 0 ${PI}" xyz="0.33 0 -0.67"/>
             <geometry>
                 <mesh filename="package://kuka_description/meshes/link1_exp.stl" scale="1 1 1"/>
@@ -59,5 +60,5 @@
         </visual>
         <collision>
-            <origin rpy="${PI / 2} 0 ${PI}" xyz="0.33 0 0.67"/>
+            <origin rpy="-${PI/2} 0 ${PI}" xyz="0.33 0 -0.67"/>
             <geometry>
                 <mesh filename="package://kuka_description/meshes/link1_exp.stl" scale="1 1 1"/>
@@ -68,5 +69,5 @@
         <xacro:default_inertial mass="0.1"/>
         <visual>
-            <origin rpy="0 0 ${PI-2*DEG2RAD}" xyz="-1.176 -0.015 0.1"/>
+            <origin rpy="0 0 ${-2*DEG2RAD}" xyz="1.176 -0.015 0.1"/>
             <geometry>
                 <mesh filename="package://kuka_description/meshes/link2_exp.stl" scale="1 1 1"/>
@@ -77,5 +78,5 @@
         </visual>
         <collision>
-            <origin rpy="0 0 ${PI}" xyz="-1.176 -0.015 0.1"/>
+            <origin rpy="0 0 ${-2*DEG2RAD}" xyz="1.176 -0.015 0.1"/>
             <geometry>
                 <mesh filename="package://kuka_description/meshes/link2_exp.stl" scale="1 1 1"/>
@@ -95,5 +96,5 @@
         </visual>
         <collision>
-            <origin rpy="0 0 ${PI/2}" xyz="-0.03 -0.15 0.01"/>
+            <origin rpy="${PI/2} 0 ${PI/2}" xyz="-0.03 -0.15 0.01"/>
             <geometry>
                 <mesh filename="package://kuka_description/meshes/link3_exp.stl" scale="1 1 1"/>
@@ -104,5 +105,5 @@
         <xacro:default_inertial mass="0.1"/>
         <visual>
-            <origin rpy="${PI/2} 0 ${PI}" xyz="0 0 1.2"/>
+            <origin rpy="-${PI/2} 0 0" xyz="0 0 -1.2"/>
             <geometry>
                 <mesh filename="package://kuka_description/meshes/link4_exp.stl" scale="1 1 1"/>
@@ -113,5 +114,5 @@
         </visual>
         <collision>
-            <origin rpy="${PI/2} 0 ${PI}" xyz="0 0 1.2"/>
+            <origin rpy="-${PI/2} 0 0" xyz="0 0 -1.2"/>
             <geometry>
                 <mesh filename="package://kuka_description/meshes/link4_exp.stl" scale="1 1 1"/>
@@ -122,5 +123,5 @@
         <xacro:default_inertial mass="0.1"/>
         <visual>
-            <origin rpy="${PI/2} 0 ${PI}" xyz="0 -0.03 -0.01"/>
+            <origin rpy="${PI/2} 0 ${PI/2}" xyz="-0.03 0 -0.01"/>
             <geometry>
                 <mesh filename="package://kuka_description/meshes/link5_exp.stl" scale="1 1 1"/>
@@ -131,5 +132,5 @@
         </visual>
         <collision>
-            <origin rpy="${PI/2} 0 ${PI}" xyz="0 -0.03 -0.01"/>
+            <origin rpy="${PI/2} 0 ${PI/2}" xyz="-0.03 0 -0.01"/>
             <geometry>
                 <mesh filename="package://kuka_description/meshes/link5_exp.stl" scale="1 1 1"/>
@@ -140,5 +141,5 @@
         <xacro:default_inertial mass="0.1"/>
         <visual>
-            <origin rpy="${PI} 0 ${PI}" xyz="0 0 -0.02"/>
+            <origin rpy="0 0 ${PI}" xyz="0 0 0.02"/>
             <geometry>
                 <mesh filename="package://kuka_description/meshes/link6_exp.stl" scale="1 1 1"/>
@@ -149,5 +150,5 @@
         </visual>
         <collision>
-            <origin rpy="${PI} 0 ${PI}" xyz="0 0 -0.02"/>
+            <origin rpy="0 0 ${PI}" xyz="0 0 0.02"/>
             <geometry>
                 <mesh filename="package://kuka_description/meshes/link6_exp.stl" scale="1 1 1"/>
@@ -165,5 +166,5 @@
         <parent link="base_link"/>
         <child link = "link_1"/>
-        <origin xyz="0 0 0"/>
+        <origin rpy="${PI} 0 0" xyz="0 0 0"/>
         <axis xyz="0 0 1"/>
         <limit lower="-${185*DEG2RAD}" upper="${185*DEG2RAD}"
@@ -173,5 +174,5 @@
         <parent link="link_1"/>
         <child link = "link_2"/>
-        <origin rpy="-${PI / 2} ${PI} 0" xyz="0.33 0 0.645"/>
+        <origin rpy="${PI / 2} 0 0" xyz="0.33 0 -0.645"/>
         <axis xyz="0 0 1"/>
         <limit lower="-${140*DEG2RAD}" upper="-${5*DEG2RAD}"
@@ -181,5 +182,5 @@
         <parent link="link_2"/>
         <child link = "link_3"/>
-        <origin rpy="0 0 ${PI}" xyz="-1.150 0 0"/>
+        <origin rpy="0 0 0" xyz="1.150 0 0"/>
         <axis xyz="0 0 1"/>
         <limit lower="-${120*DEG2RAD}" upper="${168*DEG2RAD}"
@@ -189,5 +190,5 @@
         <parent link="link_3"/>
         <child link = "link_4"/>
-        <origin rpy="${PI/2} 0 ${PI/2}" xyz="0 -0.115 0"/>
+        <origin rpy="${PI/2} 0 -${PI/2}" xyz="0 -0.115 0"/>
         <axis xyz="0 0 1"/>
         <limit lower="-${350*DEG2RAD}" upper="${350*DEG2RAD}"
@@ -197,5 +198,5 @@
         <parent link="link_4"/>
         <child link = "link_5"/>
-        <origin rpy="${PI/2} 0 ${PI}" xyz="0 0 1.220"/>
+        <origin rpy="-${PI/2} ${PI/2} 0" xyz="0 0 -1.220"/>
         <axis xyz="0 0 1"/>
         <limit lower="-${122.5*DEG2RAD}" upper="${122.5*DEG2RAD}"
@@ -205,9 +206,66 @@
         <parent link="link_5"/>
         <child link = "link_6"/>
-        <origin rpy="${PI/2} 0 ${PI}" xyz="0 0.24 0"/>
+        <origin rpy="${PI/2} 0 -${PI/2}" xyz="0.24 0 0"/>
         <axis xyz="0 0 1"/>
         <limit lower="-${350*DEG2RAD}" upper="${350*DEG2RAD}"
                effort="${effort}" velocity="${velocity}"/>
     </joint>
+    <!-- Gripper links -->
+    <link name="end_effector_link">
+        <xacro:default_inertial mass="0.1" />
+        <visual>
+            <origin xyz="0.1125 0 0" rpy="0 0 0" />
+            <geometry>
+                <box size="0.3 0.225 0.225" /> <!-- x, y, z 방향 크기 지정 -->
+            </geometry>
+            <material name="">
+                <color rgba="0 0 0 1"/>
+            </material>
+        </visual>
+        <collision>
+            <origin xyz="0.1125 0 0" rpy="0 0 0" />
+            <geometry>
+                <box size="0.3 0.225 0.225" /> <!-- x, y, z 방향 크기 지정 -->
+            </geometry>
+        </collision>
+    </link>
+    <joint name="end_effector_joint" type="revolute">
+        <parent link="link_6" />
+        <child link="end_effector_link" />
+        <origin xyz="0 0 -0.21" rpy="0 -${PI/2} ${PI/18}" />
+        <axis xyz="0 0 1"/>
+        <limit lower="0" upper="0"
+               effort="${effort}" velocity="${velocity}"/>
+    </joint>
+    <link name="drill_link">
+        <xacro:default_inertial mass="0.05" />
+        <visual>
+            <origin xyz="0 0 0.05" rpy="0 0 0" />
+            <geometry>
+                <cylinder radius="0.01" length="0.1" />
+            </geometry>
+            <material name="">
+                <color rgba="0 0 0 1"/>
+            </material>
+        </visual>
+        <collision>
+            <origin xyz="0 0 0.05" rpy="0 0 0" />
+            <geometry>
+                <cylinder radius="0.01" length="0.1" />
+            </geometry>
+        </collision>
+    </link>
+    <joint name="drill_joint" type="fixed">
+        <parent link="end_effector_link" />
+        <child link="drill_link" />
+        <origin xyz="0 0 -0.255" rpy="0 0 ${PI}" />
+    </joint>
+    <transmission name="transmission_end_effector">
+        <plugin>transmission_interface/SimpleTransmission</plugin>
+        <actuator name="end_effector_motor" role="actuator1"/>
+        <joint name="end_effector_joint" role="joint1">
+            <mechanical_reduction>1.0</mechanical_reduction>
+        </joint>
+    </transmission>
     <!-- Transmissions-->
     <xacro:default_transmission number="1"/>

File: src/kuka_description/urdf/kuka_gazebo.xacro (robot description, xacro)
@@ -7,4 +7,17 @@
         <robot_param_node>robot_state_publisher</robot_param_node>
         <parameters>$(find kuka_controller)/config/kuka_controllers.yaml</parameters>
+      </plugin>
+    </gazebo>
+    <!-- Gazebo plugin for link state publishing -->
+    <gazebo>
+      <plugin name="gazebo_ros_p3d" filename="libgazebo_ros_p3d.so">
+          <ros>
+              <namespace>gazebo</namespace>
+              <remapping>odom:=end_effector_pose</remapping> <!-- remapping을 사용하여 토픽 이름 변경 -->
+          </ros>
+          <always_on>true</always_on>
+          <update_rate>100</update_rate>
+          <body_name>end_effector_link</body_name>
+          <frame_name>world</frame_name>
       </plugin>
     </gazebo>
@@ -30,3 +43,6 @@
       <material>Gazebo/Black</material>
     </gazebo>
+    <gazebo reference="end_effector_link">
+      <material>Gazebo/Black</material>
+    </gazebo>
 </robot>

File: src/kuka_description/urdf/kuka_ros2_control.xacro (robot description, xacro)
@@ -80,4 +80,16 @@
             <state_interface name="velocity"/>
         </joint>
+        <joint name="end_effector_joint">
+            <command_interface name="position">
+            <param name="min">0</param>
+            <param name="max">0</param>
+            </command_interface>
+            <command_interface name="velocity">
+                <param name="min">0</param>
+                <param name="max">0</param>
+                </command_interface>
+            <state_interface name="position"/>
+            <state_interface name="velocity"/>
+        </joint>
     </ros2_control>
 </robot>
